File: Hardware/si4735v2.3.1.brd (EAGLE design)
At the start: 29.2 x 64.8 mm, 64 parts, among them J3 SJ2-35863A-SMT-TR, Q1 8MHz, Q4 27Mhz, U1 INFINEON_BGA427INFINEON_BGA42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, U2 STM32F103C8T6, U5 INFINEON_BGA427INFINEON_BGA42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, U6 TDA2822D, X2 SMA-142-0701-801/806

Commit message: Add files via upload
Parts:
- EEPROM: value 24C64SM -> 24C256
Changed lines of the file:
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@@
 <attribute name="VALUE" x="18.288" y="20.828" size="1.27" layer="28" rot="MR0"/>
 </element>
-<element name="EEPROM" library="microchip" library_urn="urn:adsk.eagle:library:294" package="SO-08M" package3d_urn="urn:adsk.eagle:package:20798/2" value="24C64SM" x="10.922" y="63.373" smashed="yes" rot="MR0">
+<element name="EEPROM" library="microchip" library_urn="urn:adsk.eagle:library:294" package="SO-08M" package3d_urn="urn:adsk.eagle:package:20798/2" value="24C256" x="10.922" y="63.373" smashed="yes" rot="MR0">
 <attribute name="MF" value="RAMTRON INTERNATIONAL CORP" x="-6.858" y="4.953" size="1.778" layer="28" rot="MR0" display="off"/>
 <attribute name="MPN" value="FM24C64-S" x="-6.858" y="4.953" size="1.778" layer="28" rot="MR0" display="off"/>
