File: Hardware/si4735v2.3.1.sch (EAGLE design)
At the start: 64 parts, among them J3 SJ2-35863A-SMT-TR, Q1 8MHz, Q4 27Mhz, U1 INFINEON_BGA427INFINEON_BGA42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, U2 STM32F103C8T6, U5 INFINEON_BGA427INFINEON_BGA42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, U6 TDA2822D, X2 SMA-142-0701-801/806

Commit message: Add files via upload
Parts:
- EEPROM: value 24C64SM -> 24C256
Changed lines of the file:
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@@
 <part name="J2" library="SparkFun-Connectors" library_urn="urn:adsk.eagle:library:513" deviceset="USB_MICRO-B" device="REDUCED_PASTE" package3d_urn="urn:adsk.eagle:package:38239/1"/>
 <part name="GND33" library="supply1" library_urn="urn:adsk.eagle:library:371" deviceset="GND" device=""/>
-<part name="EEPROM" library="microchip" library_urn="urn:adsk.eagle:library:294" deviceset="24*" device="SM" package3d_urn="urn:adsk.eagle:package:20798/2" technology="C64"/>
+<part name="EEPROM" library="microchip" library_urn="urn:adsk.eagle:library:294" deviceset="24*" device="SM" package3d_urn="urn:adsk.eagle:package:20798/2" technology="C64" value="24C256"/>
 <part name="GND36" library="supply1" library_urn="urn:adsk.eagle:library:371" deviceset="GND" device=""/>
 <part name="GND37" library="supply1" library_urn="urn:adsk.eagle:library:371" deviceset="GND" device=""/>
